File: AcuarioSambilSoloDC/AcuarioSambilSoloDC.kicad_pcb (KiCad board)
At the start: 2 copper layers, 154.9 x 121.9 mm, 112 parts, among them J1 BATTERY, J10 L_FOOD, J11 EC_MT, J12 PUMP 1, J13 VALVE, J14 PUMP 2, J15 PUMP 3, J16 PUMP 4, J17 PUMP 5, J18 VALVE, J19 VALVE, J2 SUPPLY, J20 VALVE, J21 VALVE, J22 VALVE, J23 VALVE, J24 KEYBOARD, J25 1WIRE, J26 RTC, J3 LCD_I2C, J4 RS485, J5 PH_RT, J6 L_RT, J7 L_SALT, J8 EC_RT, J9 L_MT, M1 SALT_DISPENSER, M2 FOOD_DISPENSER, P1 Digital, P10 CONN_01X01, P11 CONN_01X01, P12 CONN_01X01, P13 CONN_01X01, P2 Power, P3 Analog, P4 Analog, P5 PWM, P6 PWM, P7 Communication, P8 CONN_01X01, P9 CONN_01X01, SW1 PREV, SW2 MINUS, SW3 PLUS, SW4 NEXT, SW5 BACK, SW6 OK, SW8 RESET, U1 MAX485E, U2 ULN2003, U3 ULN2003, U4 ULN2003, U5 ULN2003

Commit message: Botones de funciones
Parts:
- removed G***: LOGO, nodemcu:sambilSC
Connections:
- net /B2 renamed /MB1
- net /B3 renamed /MB2
- net /B4 renamed /MB3
- net /B5 renamed /MB4
- U5 pad 16: /BUZZER -> /BZ
