File: AcuarioSambilSoloDC/AcuarioSambilSoloDC.sch (KiCad schematic (older format))
At the start: 63 parts, among them J1 BATTERY, J10 L_FOOD, J11 EC_MT, J2 SUPPLY, J24 KEYBOARD, J25 1WIRE, J26 RTC, J3 LCD_I2C, J4 RS485, J5 PH_RT, J6 L_RT, J7 L_SALT, J8 EC_RT, J9 L_MT, M1 SALT_DISPENSER, M2 FOOD_DISPENSER, P1 Digital, P10 CONN_01X01, P11 CONN_01X01, P12 CONN_01X01, P13 CONN_01X01, P2 Power, P3 Analog, P4 Analog, P5 PWM, P6 PWM, P7 Communication, P8 CONN_01X01, P9 CONN_01X01, SW1 PREV, SW2 MINUS, SW3 PLUS, SW4 NEXT, SW5 BACK, SW6 OK, SW8 RESET, U1 MAX485E, U2 ULN2003, U5 ULN2003

Commit message: funciones de actuadores
Connections:
- net labels added: MB1, MB2, MB3, MB4
- net labels removed: B2, B3, B4, B5
Changed lines of the file:
@@
 $EndComp
 Text Label 2800 2200 0    50   ~ 0
-B2
+MB1
 Text Label 3000 2200 0    50   ~ 0
-B3
+MB2
 Text Label 2450 2450 0    50   ~ 0
-B4
+MB3
 Text Label 2450 2650 0    50   ~ 0
-B5
+MB4
 Wire Wire Line
 	2600 2450 2450 2450
@@
 	2700 2200 2700 2250
 Text Label 3250 3450 0    50   ~ 0
-B2
+MB1
 Text Label 3250 3550 0    50   ~ 0
-B3
+MB2
 Text Label 3250 3650 0    50   ~ 0
-B4
+MB3
 Text Label 3250 3750 0    50   ~ 0
-B5
+MB4
 $Comp
 L conn:Conn_01x04 J7

Commit message: Botones de funciones
Changed lines of the file:
@@
 F8 "47" I R 4700 7150 50
 F9 "49" I R 4700 7250 50
-F10 "56(MOSI)" I R 4700 7350 50
+F10 "51(MOSI)" I R 4700 7350 50
 F11 "53(SS)" I R 4700 7450 50
 F12 "A15" I R 4700 5450 50
