File: AcuarioSambilSoloDC/PUMPS.sch (KiCad schematic (older format))
At the start: 48 parts, among them J12 PUMP 1, J13 VALVE, J14 PUMP 2, J15 PUMP 3, J16 PUMP 4, J17 PUMP 5, J18 VALVE, J19 VALVE, J20 VALVE, J21 VALVE, J22 VALVE, J23 VALVE, U3 ULN2003, U4 ULN2003

Commit message: Botones de funciones
Connections:
- net labels added: 51(MOSI)
- net labels removed: 56(MOSI)
Changed lines of the file:
@@
 49
 Text HLabel 4250 3900 0    50   Input ~ 0
-56(MOSI)
+51(MOSI)
 Text HLabel 4250 4000 0    50   Input ~ 0
 53(SS)
